Commit message: Fix findings from the multi-lens review of the HUNTeR replica
Model and design
- Tyre friction now reaches Gazebo (unnamed tyre collisions).
- Springs sized per axle for 1.5 Hz at both ends, so each spring unloads
  exactly at its own full droop; per-axle bump/droop limits.
- Simulated tyre is rigid: joint springs carry spring and tyre in series,
  keeping the design ride frequency and static drop.
- Axle inertia as a parallel-axis sum about its own COM (full tensor,
  mirrored for the rear axle); sensors no longer double-counted.
- Keel re-derived above the highest axle part at full bump; bumper
  collision boxes; continuous-grade estimate with drivetrain efficiency.
- Steering and linkage re-packaged: high-steer tie rod over the
  differential, upper link on a tower clear of the motor, Panhard rod
  ahead of the cover; knuckle mounting face sign fixed; brackets and
  bump stops attached to the frame.

Controller
- Command shaping keeps path curvature while ramping speed, caps speed
  for steering limits, yaw-rate, lateral acceleration and steering lag
  through the same ramp, with no windup; steering slews through the
  tie-rod linkage.
- Axle-level least-squares odometry, exact for every ICR mode, linkage
  and differential setting; odometry TF is odom -> base_footprint.
- Ackermann input sign consistent across modes, validated parameter
  updates, Twist by default, stiffer knuckle position loop in gz.

Tooling and docs
- Springs drawn at their real length (LINE_STRIP in RViz, generated
  meshes in renders); twister metrics windowed; URDF tests use the
  source tree; package dependencies completed.
- Documentation separates published facts from estimates; validation
  re-run and regenerated.

Co-Authored-By: Claude Opus 5.5 <noreply@anthropic.com>
Claude-Session: https://claude.ai/code/session_01KesnqYNaSw5wZAB7B1UQ3F

File: hunter_description/urdf/hunter.urdf.xacro (robot description, xacro)
@@ -5,6 +5,7 @@
     sim_mode        none | gz | mock | hardware   (ros2_control backend; none = no ros2_control tag)
     controllers_file  absolute path of the ros2_control controller YAML (required for sim_mode:=gz)
-    variant         2020 | 2023                     (2020 prototype 3.5 t with PTZ mast and top-view
-                                                     cameras; 2023+ armed-era 4.05 t with stereo camera)
+    variant         2020 | 2023                     (2020 prototype, 3.5 t, PTZ mast and top-view cameras;
+                                                     2023+ armed era, 3.85 t, stereo camera; 4.05 t with
+                                                     payload:=rws)
     payload         none | cargo | rws | uav_pad      (mission module on the deck)
     cargo_mass      kg, 0 = default from vehicle.yaml (payload:=cargo only)
@@ -39,11 +40,11 @@
   <xacro:property name="has_ptz" value="${sensors_on and str(variant) in V.ptz.variants and payload != 'rws'}"/>
   <xacro:property name="visual_detail" value="$(arg visual_detail)"/>
-  <xacro:include filename="$(find hunter_description)/urdf/include/common.xacro"/>
-  <xacro:include filename="$(find hunter_description)/urdf/include/chassis.xacro"/>
-  <xacro:include filename="$(find hunter_description)/urdf/include/suspension.xacro"/>
-  <xacro:include filename="$(find hunter_description)/urdf/include/sensors.xacro"/>
-  <xacro:include filename="$(find hunter_description)/urdf/include/payloads.xacro"/>
-  <xacro:include filename="$(find hunter_description)/urdf/include/ros2_control.xacro"/>
-  <xacro:include filename="$(find hunter_description)/urdf/include/gazebo.xacro"/>
+  <xacro:include filename="include/common.xacro"/>
+  <xacro:include filename="include/chassis.xacro"/>
+  <xacro:include filename="include/suspension.xacro"/>
+  <xacro:include filename="include/sensors.xacro"/>
+  <xacro:include filename="include/payloads.xacro"/>
+  <xacro:include filename="include/ros2_control.xacro"/>
+  <xacro:include filename="include/gazebo.xacro"/>
   <xacro:hunter_chassis/>
   <xacro:hunter_axle axle="front" x="${0.5 * V.chassis.wheelbase}" static_load="${V.suspension.static_load_front}"/>

File: hunter_description/urdf/include/ros2_control.xacro (robot description, xacro)
@@ -1,7 +1,7 @@
 <?xml version="1.0"?>
 <!-- ros2_control interfaces of the HUNTeR replica.
-     Steering knuckles: position command (one electric steering actuator per
-     axle drives both knuckles through the tie rod; the 4WS controller sends
-     the linkage-consistent left/right pair).
+     Steering knuckles: position command. The replica assumes one steering
+     actuator per axle driving both knuckles through the tie rod; the 4WS
+     controller sends linkage-consistent left/right pairs.
      Wheels: velocity command (axle traction motors + differentials; the
      controller emulates the electronic / locked differential).
@@ -14,7 +14,7 @@
       <hardware>
         <xacro:if value="${sim_mode == 'gz'}">
+          <!-- The knuckle position gain is a parameter of the gz_ros_control node,
+               set in hunter_control/config/controllers.yaml. -->
           <plugin>gz_ros2_control/GazeboSimSystem</plugin>
-          <!-- P gain turning knuckle position commands into joint velocity commands. -->
-          <param name="position_proportional_gain">${V.steering.sim_position_gain}</param>
         </xacro:if>
         <xacro:if value="${sim_mode == 'mock'}">

File: hunter_description/urdf/include/sensors.xacro (robot description, xacro)
@@ -1,11 +1,14 @@
 <?xml version="1.0"?>
 <!-- Sensor suite of the HUNTeR replica, generated from vehicle.yaml.
-     Published layout (see docs/DESIGN_REPORT.md):
-       2020 prototype: GPS, two lidars, 9 HD cameras = PTZ + 4 hull/side
-                       navigation cameras + 4 drive-assist cameras
-                       (front/rear driving + 2 top-view cameras on the railing)
-       2023+ armed:    2 driving + 4 perimeter cameras, RWS optics act as PTZ,
-                       stereovision cameras and extra lidars (2024)
-     Positions are reconstructions (no drawings are public).
+     Published (see docs/DESIGN_REPORT.md):
+       2020 prototype: GPS, two lidars, 9 HD cameras = PTZ + 4 hull navigation
+                       cameras + 4 drive-assist cameras; poster: front/rear driving
+                       cameras, two side cameras per side, top-view cameras on the
+                       railing (count not published), PTZ
+       2023+ armed:    2 driving + 4 perimeter cameras, RWS optics can act as PTZ;
+                       2024: additional lidars and stereovision cameras
+     Modelled here: 2 top-view cameras (so the 2020 total is 9), one stereo
+     camera for 2023 (the extra 2024 lidars are not modelled: count and position
+     unknown), and an IMU (assumed). Positions are reconstructions.
      Every camera has a <name>_optical_frame (z forward, x right, y down) used as
      the frame_id of its images. -->

File: hunter_description/urdf/include/suspension.xacro (robot description, xacro)
@@ -9,9 +9,9 @@
                   (revolute x, roll)    [axle]_axle_link
      with the two coil-overs lumped into equivalent heave and roll springs and
-     dampers (see docs/SUSPENSION_DESIGN.md):
+     dampers (see docs/MODEL.md):
        k_heave = 2 k_w            c_heave = 2 c_w
        k_roll  = 2 k_w (s/2)^2    c_roll  = 2 c_w (s/2)^2
-     with k_w, c_w the wheel-rate spring and damper per side and s the
-     spring track. The heave spring reference is set so that q = 0 at the
+     with k_w, c_w the wheel-rate spring and damper per side (per axle) and s
+     the spring track. The heave spring reference is set so that q = 0 at the
      kerb-weight static equilibrium; extra payload sags the suspension.
      The physical links (lower trailing arms, upper link, Panhard rod,
@@ -20,9 +20,16 @@
   <xacro:macro name="hunter_axle" params="axle x static_load">
     <xacro:property name="S" value="${V.suspension}"/>
-    <xacro:property name="kw" value="${S.wheel_rate}"/>
-    <xacro:property name="cw" value="${S.damping_wheel}"/>
+    <!-- Spring rates are sized per axle for the same ride frequency, so each
+         spring unloads exactly at its own full droop. -->
+    <xacro:property name="kw" value="${S.wheel_rate_front if axle == 'front' else S.wheel_rate_rear}"/>
+    <xacro:property name="cw" value="${S.damping_wheel_front if axle == 'front' else S.damping_wheel_rear}"/>
+    <xacro:property name="droop" value="${S.travel_rebound_front if axle == 'front' else S.travel_rebound_rear}"/>
+    <xacro:property name="bump" value="${S.travel_bump_front if axle == 'front' else S.travel_bump_rear}"/>
     <xacro:property name="half_s" value="${0.5 * S.spring_track}"/>
-    <xacro:property name="k_heave" value="${2.0 * kw}"/>
-    <xacro:property name="k_roll" value="${2.0 * kw * half_s * half_s + S.anti_roll_stiffness}"/>
+    <!-- The simulated tyre is rigid: these springs carry the coil springs (and
+         anti-roll bar) in series with the tyres, so the body keeps the design
+         ride frequency and static drop. -->
+    <xacro:property name="k_heave" value="${S.sim_heave_stiffness_front if axle == 'front' else S.sim_heave_stiffness_rear}"/>
+    <xacro:property name="k_roll" value="${S.sim_roll_stiffness_front if axle == 'front' else S.sim_roll_stiffness_rear}"/>
     <xacro:property name="h_rc" value="${S.roll_center_height}"/>
     <joint name="${axle}_axle_heave_joint" type="prismatic">
@@ -31,5 +38,5 @@
       <origin xyz="${x} 0 0" rpy="0 0 0"/>
       <axis xyz="0 0 1"/>
-      <limit lower="${-S.travel_rebound}" upper="${S.travel_bump}" effort="${S.joint_effort_limit}" velocity="${S.joint_velocity_limit}"/>
+      <limit lower="${-droop}" upper="${bump}" effort="${S.joint_effort_limit}" velocity="${S.joint_velocity_limit}"/>
       <dynamics damping="${2.0 * cw}" friction="${S.coulomb_friction}"/>
     </joint>
@@ -58,8 +65,13 @@
          Frame origin on the roll axis; the axle centreline is h_rc below. -->
     <link name="${axle}_axle_link">
-      <!-- The traction motor on the pinion shifts the COM toward the vehicle centre. -->
-      <xacro:property name="com_x" value="${-V.axle.com_x_toward_centre if axle == 'front' else V.axle.com_x_toward_centre}"/>
-      <xacro:inertial_tensor mass="${V.axle.mass}" xyz="${com_x} 0 ${-h_rc + V.axle.com_z_offset}"
-                             ixx="${V.axle.ixx}" iyy="${V.axle.iyy}" izz="${V.axle.izz}"/>
+      <!-- The traction motor on the pinion shifts the COM toward the vehicle centre
+           (and toward the offset differential). The rear axle is the front one
+           turned by pi about z: x and y offsets and the xz/yz products change sign. -->
+      <xacro:property name="m" value="${1 if axle == 'front' else -1}"/>
+      <xacro:property name="C" value="${V.axle.com_front}"/>
+      <xacro:property name="I" value="${V.axle.inertia_front}"/>
+      <xacro:inertial_tensor mass="${V.axle.mass}" xyz="${m * C[0]} ${m * C[1]} ${-h_rc + C[2]}"
+                             ixx="${I.ixx}" iyy="${I.iyy}" izz="${I.izz}"
+                             ixy="${I.ixy}" ixz="${m * I.ixz}" iyz="${m * I.iyz}"/>
       <xacro:if value="${visual_detail == 'mesh'}">
         <xacro:mesh_visual name="housing" file="axle_housing.stl" material="hunter_green_dark"
@@ -153,5 +165,7 @@
         </visual>
       </xacro:unless>
-      <collision name="${axle}_${side}_tyre_collision">
+      <!-- Unnamed on purpose: libsdformat only applies the link's <gazebo> friction
+           (mu1/mu2 below) to collisions it names itself. -->
+      <collision>
         <origin xyz="0 0 0" rpy="${pi/2} 0 0"/>
         <geometry><cylinder radius="${W.collision_radius}" length="${W.width}"/></geometry>

Commit message: Remove military configurations; keep the bare 2020 platform
The model now covers only the unarmed platform as first shown in 2020.

- Drop the ZMU-03 remote weapon station, cargo-mule and UAV-pad payloads
  (payloads.xacro, meshes, rws_controller, joints, renders, viewer configs)
- Drop the 2023 armed variant: variant/payload/cargo_mass arguments, the
  4.05 t armed mass and upgrade block, the variant-only stereo camera
- Remove weapon-only sources and wording from the design script, docs and
  the research archive (98 weapon/mission entries pruned, spec quotes kept)
- Rename the paint comment to olive green
- sim.launch.py: start all controllers (PTZ included) from one spawner
  with a 60 s switch timeout; the separate PTZ spawner raced the drive
  spawner and timed out under CPU-rendered sensors

The default URDF is unchanged apart from comments, so the Gazebo
validation results still apply. 86 tests pass.

Co-Authored-By: Claude Opus 5.5 <noreply@anthropic.com>
Claude-Session: https://claude.ai/code/session_01KesnqYNaSw5wZAB7B1UQ3F

File: hunter_description/urdf/hunter.urdf.xacro (robot description, xacro)
@@ -5,9 +5,4 @@
     sim_mode        none | gz | mock | hardware   (ros2_control backend; none = no ros2_control tag)
     controllers_file  absolute path of the ros2_control controller YAML (required for sim_mode:=gz)
-    variant         2020 | 2023                     (2020 prototype, 3.5 t, PTZ mast and top-view cameras;
-                                                     2023+ armed era, 3.85 t, stereo camera; 4.05 t with
-                                                     payload:=rws)
-    payload         none | cargo | rws | uav_pad      (mission module on the deck)
-    cargo_mass      kg, 0 = default from vehicle.yaml (payload:=cargo only)
     sensors         true | false                    (lidars, cameras, GNSS, IMU, PTZ)
     camera_sensors  true | false                    (Gazebo camera sensors; frames are always present)
@@ -21,7 +16,4 @@
   <xacro:arg name="sim_mode" default="none"/>
   <xacro:arg name="controllers_file" default=""/>
-  <xacro:arg name="variant" default="2020"/>
-  <xacro:arg name="payload" default="none"/>
-  <xacro:arg name="cargo_mass" default="0"/>
   <xacro:arg name="sensors" default="true"/>
   <xacro:arg name="camera_sensors" default="true"/>
@@ -31,12 +23,9 @@
   <xacro:property name="V" value="${xacro.load_yaml('$(arg vehicle_file)')}"/>
   <xacro:property name="sim_mode" value="$(arg sim_mode)"/>
-  <!-- Normalise booleans; compare the variant with str(variant) (xacro turns '2020' into an int). -->
-  <xacro:property name="variant" value="$(arg variant)"/>
-  <xacro:property name="payload" value="$(arg payload)"/>
-  <xacro:property name="cargo_mass" value="$(arg cargo_mass)"/>
+  <!-- Normalise booleans. -->
   <xacro:property name="sensors_on" value="${'$(arg sensors)'.lower() in ('true', '1')}"/>
   <xacro:property name="camera_sensors" value="${'$(arg camera_sensors)'.lower() in ('true', '1')}"/>
   <xacro:property name="lidar_resolution" value="$(arg lidar_resolution)"/>
-  <xacro:property name="has_ptz" value="${sensors_on and str(variant) in V.ptz.variants and payload != 'rws'}"/>
+  <xacro:property name="has_ptz" value="${sensors_on}"/>
   <xacro:property name="visual_detail" value="$(arg visual_detail)"/>
   <xacro:include filename="include/common.xacro"/>
@@ -44,5 +33,4 @@
   <xacro:include filename="include/suspension.xacro"/>
   <xacro:include filename="include/sensors.xacro"/>
-  <xacro:include filename="include/payloads.xacro"/>
   <xacro:include filename="include/ros2_control.xacro"/>
   <xacro:include filename="include/gazebo.xacro"/>
@@ -53,5 +41,4 @@
     <xacro:hunter_sensors/>
   </xacro:if>
-  <xacro:hunter_payload payload="${payload}"/>
   <xacro:unless value="${sim_mode == 'none'}">
     <xacro:hunter_ros2_control sim_mode="${sim_mode}"/>

File: hunter_description/urdf/include/common.xacro (robot description, xacro)
@@ -3,5 +3,5 @@
 <robot xmlns:xacro="http://www.ros.org/wiki/xacro">
   <!-- ===================================================== materials -->
-  <!-- Polish Army green (approx. RAL 6031 / "khaki-green" field finish). -->
+  <!-- Olive green body paint (approx. RAL 6031). -->
   <material name="hunter_green"><color rgba="0.247 0.290 0.180 1.0"/></material>
   <material name="hunter_green_dark"><color rgba="0.180 0.212 0.137 1.0"/></material>

File: hunter_description/urdf/include/ros2_control.xacro (robot description, xacro)
@@ -79,8 +79,4 @@
         <xacro:position_iface name="ptz_tilt_joint" lo="${-radians(V.ptz.tilt_max_deg)}" hi="${-radians(V.ptz.tilt_min_deg)}"/>
       </xacro:if>
-      <xacro:if value="${payload == 'rws'}">
-        <xacro:position_iface name="rws_yaw_joint" lo="${-1e9}" hi="${1e9}"/>
-        <xacro:position_iface name="rws_pitch_joint" lo="${radians(V.payloads.rws.pitch_min_deg)}" hi="${radians(V.payloads.rws.pitch_max_deg)}"/>
-      </xacro:if>
     </ros2_control>
   </xacro:macro>

File: hunter_description/urdf/include/sensors.xacro (robot description, xacro)
@@ -6,9 +6,6 @@
                        cameras, two side cameras per side, top-view cameras on the
                        railing (count not published), PTZ
-       2023+ armed:    2 driving + 4 perimeter cameras, RWS optics can act as PTZ;
-                       2024: additional lidars and stereovision cameras
-     Modelled here: 2 top-view cameras (so the 2020 total is 9), one stereo
-     camera for 2023 (the extra 2024 lidars are not modelled: count and position
-     unknown), and an IMU (assumed). Positions are reconstructions.
+     Modelled here: 2 top-view cameras (so the total is 9) and an IMU (assumed).
+     Positions are reconstructions.
      Every camera has a <name>_optical_frame (z forward, x right, y down) used as
      the frame_id of its images. -->
@@ -109,29 +106,4 @@
     </xacro:if>
   </xacro:macro>
-  <xacro:macro name="hunter_stereo" params="s">
-    <link name="${s['name']}_link">
-      <xacro:inertial_box mass="0.5" x="0.04" y="0.18" z="0.05"><origin xyz="-0.02 0 0"/></xacro:inertial_box>
-      <xacro:mesh_visual file="stereo_camera.stl" material="sensor_black"/>
-    </link>
-    <joint name="${s['name']}_joint" type="fixed">
-      <parent link="base_link"/>
-      <child link="${s['name']}_link"/>
-      <origin xyz="${s['xyz'][0]} ${s['xyz'][1]} ${s['xyz'][2]}" rpy="${s['rpy'][0]} ${s['rpy'][1]} ${s['rpy'][2]}"/>
-    </joint>
-    <xacro:macro name="stereo_eye" params="eye y">
-      <link name="${s['name']}_${eye}_link"/>
-      <joint name="${s['name']}_${eye}_joint" type="fixed">
-        <parent link="${s['name']}_link"/>
-        <child link="${s['name']}_${eye}_link"/>
-        <origin xyz="0.01 ${y} 0" rpy="0 0 0"/>
-      </joint>
-      <xacro:optical_frame name="${s['name']}_${eye}"/>
-      <xacro:if value="${camera_sensors}">
-        <xacro:gz_camera name="${s['name']}_${eye}" hfov="${s['hfov_deg']}" width="${s['width']}" height="${s['height']}" rate="${s['rate']}" far="60.0"/>
-      </xacro:if>
-    </xacro:macro>
-    <xacro:stereo_eye eye="left" y="${s['baseline'] / 2}"/>
-    <xacro:stereo_eye eye="right" y="${-s['baseline'] / 2}"/>
-  </xacro:macro>
   <!-- ============================================================== GNSS -->
   <xacro:macro name="hunter_navsat" params="s">
@@ -265,11 +237,8 @@
     <xacro:if value="${len(items) > 0}">
       <xacro:property name="s" value="${items[0]}"/>
-      <xacro:if value="${str(variant) in s['variants']}">
-        <xacro:if value="${s['type'] == 'lidar'}"><xacro:hunter_lidar s="${s}"/></xacro:if>
-        <xacro:if value="${s['type'] == 'camera'}"><xacro:hunter_camera s="${s}"/></xacro:if>
-        <xacro:if value="${s['type'] == 'stereo'}"><xacro:hunter_stereo s="${s}"/></xacro:if>
-        <xacro:if value="${s['type'] == 'navsat'}"><xacro:hunter_navsat s="${s}"/></xacro:if>
-        <xacro:if value="${s['type'] == 'imu'}"><xacro:hunter_imu s="${s}"/></xacro:if>
-      </xacro:if>
+      <xacro:if value="${s['type'] == 'lidar'}"><xacro:hunter_lidar s="${s}"/></xacro:if>
+      <xacro:if value="${s['type'] == 'camera'}"><xacro:hunter_camera s="${s}"/></xacro:if>
+      <xacro:if value="${s['type'] == 'navsat'}"><xacro:hunter_navsat s="${s}"/></xacro:if>
+      <xacro:if value="${s['type'] == 'imu'}"><xacro:hunter_imu s="${s}"/></xacro:if>
       <xacro:sensor_list items="${items[1:]}"/>
     </xacro:if>
@@ -277,7 +246,5 @@
   <xacro:macro name="hunter_sensors">
     <xacro:sensor_list items="${V.sensors}"/>
-    <xacro:if value="${str(variant) in V.ptz.variants and payload != 'rws'}">
-      <xacro:hunter_ptz/>
-    </xacro:if>
+    <xacro:hunter_ptz/>
   </xacro:macro>
 </robot>
