Commit message: Reshape the hull to the photographed vehicle
User-supplied update (see CHANGELOG.md): closed, faceted body measured
against the 1 m wheel from 2023-2025 photos, with sensor band, lamps,
tow bars and shackles, wheel-arch trims, louvred tub and stepped rear
deck; 16 collision boxes (optionally pitched) following the new hull;
sensors moved onto the hull; PTZ camera removed; new
tools/check_clearance.py run by the URDF tests. Running gear,
suspension, steering, drivetrain and mass budget are unchanged.

Co-Authored-By: Claude Opus 5.5 <noreply@anthropic.com>
Claude-Session: https://claude.ai/code/session_01KesnqYNaSw5wZAB7B1UQ3F

File: hunter_description/urdf/hunter.urdf.xacro (robot description, xacro)
@@ -5,5 +5,5 @@
     sim_mode        none | gz | mock | hardware   (ros2_control backend; none = no ros2_control tag)
     controllers_file  absolute path of the ros2_control controller YAML (required for sim_mode:=gz)
-    sensors         true | false                    (lidars, cameras, GNSS, IMU, PTZ)
+    sensors         true | false                    (lidars, cameras, GNSS, IMU)
     camera_sensors  true | false                    (Gazebo camera sensors; frames are always present)
     lidar_resolution  0..1 fraction of the lidar's native horizontal samples simulated
@@ -27,5 +27,4 @@
   <xacro:property name="camera_sensors" value="${'$(arg camera_sensors)'.lower() in ('true', '1')}"/>
   <xacro:property name="lidar_resolution" value="$(arg lidar_resolution)"/>
-  <xacro:property name="has_ptz" value="${sensors_on}"/>
   <xacro:property name="visual_detail" value="$(arg visual_detail)"/>
   <xacro:include filename="include/common.xacro"/>

File: hunter_description/urdf/include/chassis.xacro (robot description, xacro)
@@ -1,11 +1,13 @@
 <?xml version="1.0"?>
-<!-- Hull / sprung mass of the HUNTeR replica. -->
+<!-- Hull / sprung mass of the HUNTeR replica.
+     Shape: the closed, faceted hull of the 2023-2025 vehicle (see docs/MODEL.md). -->
 <robot xmlns:xacro="http://www.ros.org/wiki/xacro">
-  <!-- Recursive helper: one <collision> per [cx, cy, cz, sx, sy, sz] entry. -->
+  <!-- Recursive helper: one <collision> per [cx, cy, cz, sx, sy, sz, pitch] entry
+       (pitch about y: the glacis and the rear lip are inclined plates). -->
   <xacro:macro name="box_collisions" params="boxes idx:=0">
     <xacro:if value="${len(boxes) > 0}">
       <xacro:property name="b" value="${boxes[0]}"/>
       <collision name="hull_collision_${idx}">
-        <origin xyz="${b[0]} ${b[1]} ${b[2]}" rpy="0 0 0"/>
+        <origin xyz="${b[0]} ${b[1]} ${b[2]}" rpy="0 ${b[6] if len(b) > 6 else 0} 0"/>
         <geometry><box size="${b[3]} ${b[4]} ${b[5]}"/></geometry>
       </collision>
@@ -17,5 +19,5 @@
       <xacro:property name="b" value="${boxes[0]}"/>
       <visual name="hull_box_${idx}">
-        <origin xyz="${b[0]} ${b[1]} ${b[2]}" rpy="0 0 0"/>
+        <origin xyz="${b[0]} ${b[1]} ${b[2]}" rpy="0 ${b[6] if len(b) > 6 else 0} 0"/>
         <geometry><box size="${b[3]} ${b[4]} ${b[5]}"/></geometry>
         <material name="${material}"/>
@@ -44,6 +46,13 @@
       <xacro:if value="${visual_detail == 'mesh'}">
         <xacro:mesh_visual name="hull" file="hull.stl" material="hunter_green"/>
+        <xacro:mesh_visual name="hull_black" file="hull_black.stl" material="hull_black"/>
+        <xacro:mesh_visual name="hull_trim" file="hull_trim.stl" material="trim_anthracite"/>
+        <xacro:mesh_visual name="hull_plates" file="hull_plates.stl" material="hunter_green_light"/>
+        <xacro:mesh_visual name="hull_glass" file="hull_glass.stl" material="glass"/>
         <xacro:mesh_visual name="hull_details" file="hull_details.stl" material="hunter_green_dark"/>
         <xacro:mesh_visual name="hull_steel" file="hull_steel.stl" material="steel_dark"/>
+        <xacro:mesh_visual name="hull_shackles" file="hull_shackles.stl" material="chrome"/>
+        <xacro:mesh_visual name="hull_shackle_pins" file="hull_shackle_pins.stl" material="pin_blue"/>
+        <xacro:mesh_visual name="hull_tiedowns" file="hull_tiedowns.stl" material="tiedown_orange"/>
         <xacro:mesh_visual name="lamps_white" file="lamps_white.stl" material="lamp_white"/>
         <xacro:mesh_visual name="lamps_amber" file="lamps_amber.stl" material="lamp_amber"/>

File: hunter_description/urdf/include/common.xacro (robot description, xacro)
@@ -3,9 +3,16 @@
 <robot xmlns:xacro="http://www.ros.org/wiki/xacro">
   <!-- ===================================================== materials -->
-  <!-- Olive green body paint (approx. RAL 6031). -->
-  <material name="hunter_green"><color rgba="0.247 0.290 0.180 1.0"/></material>
-  <material name="hunter_green_dark"><color rgba="0.180 0.212 0.137 1.0"/></material>
+  <!-- Matte grey-olive body paint as photographed (NATO-green family). -->
+  <material name="hunter_green"><color rgba="0.262 0.302 0.235 1.0"/></material>
+  <material name="hunter_green_dark"><color rgba="0.200 0.232 0.180 1.0"/></material>
+  <material name="hunter_green_light"><color rgba="0.330 0.370 0.290 1.0"/></material>
+  <!-- Front sensor band, frame tunnel, tray floor. -->
+  <material name="hull_black"><color rgba="0.060 0.060 0.065 1.0"/></material>
+  <!-- Wheel-arch trims and the sloped rear lip. -->
+  <material name="trim_anthracite"><color rgba="0.170 0.180 0.180 1.0"/></material>
+  <material name="pin_blue"><color rgba="0.100 0.300 0.800 1.0"/></material>
+  <material name="tiedown_orange"><color rgba="0.900 0.450 0.080 1.0"/></material>
   <material name="tyre_black"><color rgba="0.055 0.055 0.055 1.0"/></material>
-  <material name="rim_dark"><color rgba="0.200 0.220 0.170 1.0"/></material>
+  <material name="rim_dark"><color rgba="0.100 0.100 0.100 1.0"/></material>
   <material name="steel"><color rgba="0.420 0.430 0.440 1.0"/></material>
   <material name="steel_dark"><color rgba="0.250 0.255 0.260 1.0"/></material>

File: hunter_description/urdf/include/ros2_control.xacro (robot description, xacro)
@@ -75,8 +75,4 @@
       <xacro:passive_iface name="rear_axle_heave_joint"/>
       <xacro:passive_iface name="rear_axle_roll_joint"/>
-      <xacro:if value="${has_ptz}">
-        <xacro:position_iface name="ptz_pan_joint" lo="${-1e9}" hi="${1e9}"/>
-        <xacro:position_iface name="ptz_tilt_joint" lo="${-radians(V.ptz.tilt_max_deg)}" hi="${-radians(V.ptz.tilt_min_deg)}"/>
-      </xacro:if>
     </ros2_control>
   </xacro:macro>

File: hunter_description/urdf/include/sensors.xacro (robot description, xacro)
@@ -6,6 +6,9 @@
                        cameras, two side cameras per side, top-view cameras on the
                        railing (count not published), PTZ
-     Modelled here: 2 top-view cameras (so the total is 9) and an IMU (assumed).
-     Positions are reconstructions.
+     Modelled here: 8 fixed cameras (2 top-view, count not published) and an IMU
+     (assumed). The 2020 PTZ mast is not modelled: the photographed vehicles carry
+     a weapon station or payload with its own sensor head there instead.
+     Positions are reconstructions on the photographed 2023-2025 hull (no railing:
+     the top-view cameras sit on the deck-corner outriggers / a rear deck post).
      Every camera has a <name>_optical_frame (z forward, x right, y down) used as
      the frame_id of its images. -->
@@ -167,70 +170,4 @@
     </gazebo>
   </xacro:macro>
-  <!-- =============================================================== PTZ -->
-  <xacro:macro name="hunter_ptz">
-    <xacro:property name="P" value="${V.ptz}"/>
-    <link name="ptz_mast_link">
-      <xacro:inertial_box mass="6.0" x="0.18" y="0.18" z="${P.mast_height}"><origin xyz="0 0 ${P.mast_height / 2}"/></xacro:inertial_box>
-      <xacro:mesh_visual file="ptz_mast.stl" material="hunter_green_dark"/>
-    </link>
-    <joint name="ptz_mast_joint" type="fixed">
-      <parent link="base_link"/>
-      <child link="ptz_mast_link"/>
-      <origin xyz="${P.mount_xyz[0]} ${P.mount_xyz[1]} ${P.mount_xyz[2]}" rpy="0 0 0"/>
-    </joint>
-    <link name="ptz_pan_link">
-      <xacro:inertial_box mass="2.0" x="0.12" y="0.26" z="0.22"><origin xyz="0 0 0.11"/></xacro:inertial_box>
-      <xacro:mesh_visual file="ptz_yoke.stl" material="sensor_grey"/>
-    </link>
-    <joint name="ptz_pan_joint" type="continuous">
-      <parent link="ptz_mast_link"/>
-      <child link="ptz_pan_link"/>
-      <origin xyz="0 0 ${P.mast_height}" rpy="0 0 0"/>
-      <axis xyz="0 0 1"/>
-      <limit effort="50" velocity="1.5"/>
-      <dynamics damping="2.0"/>
-    </joint>
-    <link name="ptz_camera_link">
-      <xacro:inertial_box mass="3.0" x="${P.head_size}" y="0.2" z="0.14"><origin xyz="0 0 0"/></xacro:inertial_box>
-      <xacro:mesh_visual file="ptz_head.stl" material="sensor_grey"/>
-    </link>
-    <joint name="ptz_tilt_joint" type="revolute">
-      <parent link="ptz_pan_link"/>
-      <child link="ptz_camera_link"/>
-      <origin xyz="0 0 0.15" rpy="0 0 0"/>
-      <axis xyz="0 1 0"/>
-      <!-- +y axis: positive tilt looks down -->
-      <limit lower="${-radians(P.tilt_max_deg)}" upper="${-radians(P.tilt_min_deg)}" effort="50" velocity="1.0"/>
-      <dynamics damping="2.0"/>
-    </joint>
-    <link name="ptz_lens_link"/>
-    <joint name="ptz_lens_joint" type="fixed">
-      <parent link="ptz_camera_link"/>
-      <child link="ptz_lens_link"/>
-      <origin xyz="${P.head_size / 2 + 0.02} 0.04 0" rpy="0 0 0"/>
-    </joint>
-    <link name="ptz_camera_optical_frame"/>
-    <joint name="ptz_camera_optical_joint" type="fixed">
-      <parent link="ptz_lens_link"/>
-      <child link="ptz_camera_optical_frame"/>
-      <origin xyz="0 0 0" rpy="${-pi/2} 0 ${-pi/2}"/>
-    </joint>
-    <xacro:if value="${camera_sensors}">
-      <gazebo reference="ptz_lens_link">
-        <sensor name="ptz_camera" type="camera">
-          <always_on>true</always_on>
-          <update_rate>15</update_rate>
-          <topic>ptz_camera/image_raw</topic>
-          <gz_frame_id>ptz_camera_optical_frame</gz_frame_id>
-          <camera>
-            <camera_info_topic>ptz_camera/camera_info</camera_info_topic>
-            <horizontal_fov>${radians(P.hfov_wide_deg)}</horizontal_fov>
-            <image><width>1280</width><height>720</height><format>R8G8B8</format></image>
-            <clip><near>0.1</near><far>1000</far></clip>
-          </camera>
-        </sensor>
-      </gazebo>
-    </xacro:if>
-  </xacro:macro>
   <!-- ============================================================ driver -->
   <xacro:macro name="sensor_list" params="items">
@@ -246,5 +183,4 @@
   <xacro:macro name="hunter_sensors">
     <xacro:sensor_list items="${V.sensors}"/>
-    <xacro:hunter_ptz/>
   </xacro:macro>
 </robot>
